Commit message: Patch issues with urdf
Former-commit-id: 001ab21eb38c8d6b299986fdf823b09d32cd8b90 [formerly 8c5b01f7f24f8e259d40703d81c7bb96eef66702]
Former-commit-id: a30aac3de7678df3d68f0ba3e3b8ed426dbec904

File: kobuki_description/urdf/kobuki.urdf.xacro (robot description, xacro)
@@ -227,7 +227,7 @@
 	    <visual>
 		    <origin xyz="0 0 0" rpy="0 0 0"/>
-		    <geometry>
+		    <!-- <geometry>
 			    <mesh filename="package://hokuyo/meshes/hokuyo.dae"/>
-		    </geometry>
+		    </geometry> -->
 	    </visual>
     </link>
